File: hardware/board/microcontroller-unit.kicad_sch (KiCad schematic)
At the start: 1 part, among them U1 RP2040

Commit message: update microcontroller
Parts:
- removed U1: RP2040, Package_DFN_QFN:QFN-56-1EP_7x7mm_P0.4mm_EP3.2x3.2mm, symbol MCU_RaspberryPi:RP2040
- added C1, C10: 1uF, Capacitor_SMD:C_01005_0402Metric, symbol Device:C
- added C11, C12, C17, C2, C3, C4, C5, C6, C7, C8, C9: 0.1uF, Capacitor_SMD:C_01005_0402Metric, symbol Device:C
- added C13, C14: 10uF, Capacitor_SMD:C_0603_1608Metric, symbol Device:C
- added C15, C16: 33pF, Capacitor_SMD:C_01005_0402Metric, symbol Device:C
- added J1: USB_C_Receptacle_USB2.0_14P, Connector_USB:USB_C_Receptacle_HRO_TYPE-C-31-M-12, symbol Connector:USB_C_Receptacle_USB2.0_14P
- added R3, R4: 27, Resistor_SMD:R_0402_1005Metric, symbol Device:R
- added R3, R4: 5.1K, Resistor_SMD:R_0402_1005Metric, symbol Device:R
- added R5, R7: 1K, Resistor_SMD:R_0402_1005Metric, symbol Device:R
- added R6: 10K, Resistor_SMD:R_0402_1005Metric, symbol Device:R
- added SW1: SW_Push, Button_Switch_SMD:SW_Push_SPST_NO_Alps_SKRK, symbol Switch:SW_Push
- added U2: RP2040, Package_DFN_QFN:QFN-56-1EP_7x7mm_P0.4mm_EP3.2x3.2mm, symbol MCU_RaspberryPi:RP2040
- added U2: MCP1700x-330xxTT, Package_TO_SOT_SMD:SOT-23, symbol Regulator_Linear:MCP1700x-330xxTT
- added U3: W25Q16JVZPIQ TR, W25Q16JVUXIQ_TR:IC_W25Q16JVUXIQ_TR, symbol Memory_Flash:W25Q128JVS
- added Y1: 12 MHz, Crystal:Crystal_SMD_3225-4Pin_3.2x2.5mm, symbol Device:Crystal_GND24
Connections:
- net GND: now also C1.2, C10.2, C11.2, C12.2, C13.2, C14.2, C15.1, C16.1, C17.2, C2.2, C3.2, C4.2, C5.2, C6.2, C7.2, C8.2, C9.2, J1.A1 (GND), J1.A12 (GND), J1.B1 (GND), J1.B12 (GND), J1.S1 (SHIELD), R3.2, R4.2, SW1.1, U2.1 (GND), U2.19 (TESTEN), U2.57 (GND), U3.4 (GND), Y1.2, Y1.4
- new net: R7.1, SW1.2
- new net: C16.2, R5.1, Y1.1
- new net: R3.2, U2.47 (USB_DP)
- new net: R4.2, U2.46 (USB_DM)
- new net: J1.A5 (CC1), R3.1
- new net: J1.B5 (CC2), R4.1
- new net +1V1: C10.1, C11.1, C12.1, U2.23 (DVDD), U2.45 (VREG_VOUT), U2.50 (DVDD)
- new net +3V3: C1.1, C13.1, C17.1, C2.1, C3.1, C4.1, C5.1, C6.1, C7.1, C8.1, C9.1, R6.1, U2.1 (IOVDD), U2.10 (IOVDD), U2.2 (VO), U2.22 (IOVDD), U2.33 (IOVDD), U2.42 (IOVDD), U2.43 (ADC_AVDD), U2.44 (VREG_IN), U2.48 (USB_VDD), U2.49 (IOVDD), U3.8 (VCC)
- new net GPIO0: U2.2 (GPIO0)
- new net GPIO1: U2.3 (GPIO1)
- new net GPIO10: U2.13 (GPIO10)
- new net GPIO11: U2.14 (GPIO11)
- new net GPIO12: U2.15 (GPIO12)
- new net GPIO13: U2.16 (GPIO13)
- new net GPIO14: U2.17 (GPIO14)
- new net GPIO15: U2.18 (GPIO15)
- new net GPIO16: U2.27 (GPIO16)
- new net GPIO17: U2.28 (GPIO17)
- new net GPIO18: U2.29 (GPIO18)
- new net GPIO19: U2.30 (GPIO19)
- new net GPIO2: U2.4 (GPIO2)
- new net GPIO20: U2.31 (GPIO20)
- new net GPIO21: U2.32 (GPIO21)
- new net GPIO22: U2.34 (GPIO22)
- new net GPIO23: U2.35 (GPIO23)
- new net GPIO24: U2.36 (GPIO24)
- new net GPIO25: U2.37 (GPIO25)
- new net GPIO26_ADC0: U2.38 (GPIO26_ADC0)
- new net GPIO27_ADC1: U2.39 (GPIO27_ADC1)
- new net GPIO28_ADC2: U2.40 (GPIO28_ADC2)
- new net GPIO29_ADC3: U2.41 (GPIO29_ADC3)
- new net GPIO3: U2.5 (GPIO3)
- new net GPIO4: U2.6 (GPIO4)
- new net GPIO5: U2.7 (GPIO5)
- new net GPIO6: U2.8 (GPIO6)
- new net GPIO7: U2.9 (GPIO7)
- new net GPIO8: U2.11 (GPIO8)
- new net GPIO9: U2.12 (GPIO9)
- new net QSPI_SCLK: U2.52 (QSPI_SCLK), U3.6 (CLK)
- new net QSPI_SD0: U2.53 (QSPI_SD0), U3.5 (DI/IO_{0})
- new net QSPI_SD1: U2.55 (QSPI_SD1), U3.2 (DO/IO_{1})
- new net QSPI_SD2: U2.54 (QSPI_SD2), U3.3 (~{WP}/IO_{2})
- new net QSPI_SD3: U2.51 (QSPI_SD3), U3.7 (~{HOLD}/~{RESET}/IO_{3})
- new net QSPI_SS: R6.2, R7.2, U2.56 (QSPI_SS), U3.1 (~{CS})
- new net RUN: U2.26 (RUN)
- new net SWCLK: U2.24 (SWCLK)
- new net SWD: U2.25 (SWD)
- new net USB_D+: J1.A6 (D+), J1.B6 (D+), R3.1
- new net USB_D-: J1.A7 (D-), J1.B7 (D-), R4.1
- new net VBUS: C14.1, J1.A4 (VBUS), J1.A9 (VBUS), J1.B4 (VBUS), J1.B9 (VBUS), U2.3 (VI)
- new net XIN: C15.2, U2.20 (XIN), Y1.3
- new net XOUT: R5.2, U2.21 (XOUT)
Other:
- note added: "MOVE POWER MANAGEMENT TO POWER MANAGEMENT"
